File: HBridge.kicad_pcb (KiCad board)
At the start: 2 copper layers, 30.4 x 28.7 mm, 28 parts, among them Q1 DMG2301L, Q2 DMG3402L, Q3 DMG2301L, Q4 DMG3402L, U1 74LVC1GU04DRL, U10 LT1762, U2 74AHC1G08, U3 74AHC1G08, U4 74AHC1G08, U5 74AHC1G08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

Commit message: Add files via upload
Parts:
- moved C9 3.33 mm to (179.3, 71.6), turned to 90 degrees
- moved C2 1.26 mm to (186.5, 70.5)
- moved C1 0.80 mm to (186.7, 93.4), turned to -90 degrees
Routing:
- net +3.3V: track 55.6 -> 40.1 mm
- net GND: track 28.4 -> 24.5 mm, vias 15 -> 13
- net Net-(U5-Pad1): track 6.04 -> 8.92 mm, vias 2 -> 0
- net /Enable: track 36.5 -> 34.6 mm
- net Net-(U1-Pad4): track 5.92 -> 7.34 mm, vias 0 -> 2

Commit message: Add files via upload
Routing:
- net GND: track 24.5 -> 28.0 mm, vias 13 -> 16
Changed lines of the file:
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@@
 		(tags "SOT TO_SOT_SMD")
 		(property "Reference" "U5"
-			(at -1.2875 -2.35 0)
+			(at -1.5875 -2.55 0)
 			(layer "F.SilkS")
 			(effects
@@
 	)
 	(segment
+		(start 186.7 94.175)
+		(end 187.875 94.175)
+		(width 0.5)
+		(layer "F.Cu")
+		(net 1)
+	)
+	(segment
 		(start 180.5 86.1)
 		(end 180.3375 86.2625)
@@
 	)
 	(segment
+		(start 181.6 71.4)
+		(end 181.6 70.7)
+		(width 0.127)
+		(layer "F.Cu")
+		(net 1)
+	)
+	(segment
 		(start 187.8 69.7)
 		(end 187.775 69.725)
@@
 	)
 	(segment
+		(start 187.875 94.175)
+		(end 187.9 94.2)
+		(width 0.5)
+		(layer "F.Cu")
+		(net 1)
+	)
+	(segment
 		(start 181.5875 75.825)
 		(end 181.5875 76.6875)
@@
 	)
 	(segment
+		(start 179.3 70.825)
+		(end 178.225 70.825)
+		(width 0.5)
+		(layer "F.Cu")
+		(net 1)
+	)
+	(segment
 		(start 182.5125 92.6)
 		(end 182.5125 91.9125)
@@
 	)
 	(segment
-		(start 182.1 71.274)
-		(end 182.2 71.274)
-		(width 0.5)
-		(layer "F.Cu")
-		(net 1)
-	)
-	(segment
 		(start 176 90.975)
 		(end 177.275 90.975)
@@
 	)
 	(segment
+		(start 182.2 71.4)
+		(end 181.6 71.4)
+		(width 0.127)
+		(layer "F.Cu")
+		(net 1)
+	)
+	(segment
 		(start 183.5 72.95)
 		(end 183.575 72.875)
@@
 	)
 	(segment
+		(start 178.2 70.8)
+		(end 178.225 70.825)
+		(width 0.5)
+		(layer "F.Cu")
+		(net 1)
+	)
+	(segment
 		(start 183.025 75.825)
 		(end 183.3 76.1)
@@
 		(at 187.775 69.725)
 		(size 0.6)
-		(drill 0.3)
+		(drill 0.2)
+		(layers "F.Cu" "B.Cu")
+		(net 1)
+	)
+	(via
+		(at 178.225 70.825)
+		(size 0.6)
+		(drill 0.2)
 		(layers "F.Cu" "B.Cu")
 		(net 1)
@@
 	)
 	(via
+		(at 181.6 70.7)
+		(size 0.6)
+		(drill 0.2)
+		(layers "F.Cu" "B.Cu")
+		(net 1)
+	)
+	(via
 		(at 188.2 87.4)
 		(size 0.6)
@@
 	)
 	(via
+		(at 187.9 94.2)
+		(size 0.6)
+		(drill 0.2)
+		(layers "F.Cu" "B.Cu")
+		(net 1)
+	)
+	(via
 		(at 183.5 73.2)
 		(size 0.6)
@@
 		(at 182.7 74.3)
 		(size 0.6)
-		(drill 0.3)
+		(drill 0.2)
 		(layers "F.Cu" "B.Cu")
 		(net 3)
@@
 		(at 182.7 69.5)
 		(size 0.6)
-		(drill 0.3)
+		(drill 0.2)
 		(layers "F.Cu" "B.Cu")
 		(net 3)
@@
 		(at 187.1 90.4)
 		(size 0.6)
-		(drill 0.3)
+		(drill 0.2)
 		(layers "F.Cu" "B.Cu")
 		(net 14)
@@
 		(at 184.5 91.8)
 		(size 0.6)
-		(drill 0.3)
+		(drill 0.2)
 		(layers "F.Cu" "B.Cu")
 		(net 14)
@@
 	)
 	(zone
-		(net 3)
-		(net_name "+3.3V")
+		(net 20)
+		(net_name "/Input2")
 		(layer "F.Cu")
 		(name "$teardrop_padvia$")
 		(hatch none 0.1)
-		(priority 30000)
+		(priority 30005)
 		(attr
 			(teardrop
@@
 		(polygon
 			(pts
-				(xy 190.749 76.705764) (xy 190.249 76.705764) (xy 190.155764 77.241473) (xy 190.45 77.301) (xy 190.744236 77.358527)
+				(xy 181.5635 72.605764) (xy 181.4365 72.605764) (xy 181.250559 73.033329) (xy 181.5 73.201) (xy 181.749441 73.033329)
 			)
 		)
@@
 		(polygon
 			(pts
-				(xy 177.1 88.8) (xy 174.9 88.8) (xy 174.9 97.2) (xy 188.8 97.2) (xy 188.8 88.4) (xy 182.141551 88.4)
+				(xy 177.1 88.8) (xy 174.9 88.8) (xy 174.9 97.2) (xy 190 97.2) (xy 190 88.4) (xy 182.141551 88.4)
 				(xy 184.433177 93.888436) (xy 179.016777 93.830241) (xy 179.2 88.7)
 			)
@@
 	)
 	(zone
-		(net 7)
-		(net_name "/MotorConnect2")
+		(net 3)
+		(net_name "+3.3V")
 		(layer "F.Cu")
 		(name "$teardrop_padvia$")
 		(hatch none 0.1)
-		(priority 30001)
+		(priority 30000)
 		(attr
 			(teardrop
@@
 		(polygon
 			(pts
-				(xy 183.25 82.194236) (xy 183.75 82.194236) (xy 183.794236 81.658527) (xy 183.5 81.599) (xy 183.205764 81.658527)
+				(xy 190.749 76.705764) (xy 190.249 76.705764) (xy 190.155764 77.241473) (xy 190.45 77.301) (xy 190.744236 77.358527)
 			)
 		)
 	)
 	(zone
-		(net 20)
-		(net_name "/Input2")
+		(net 7)
+		(net_name "/MotorConnect2")
 		(layer "F.Cu")
 		(name "$teardrop_padvia$")
 		(hatch none 0.1)
-		(priority 30005)
+		(priority 30001)
 		(attr
 			(teardrop
@@
 		(polygon
 			(pts
-				(xy 181.5635 72.605764) (xy 181.4365 72.605764) (xy 181.250559 73.033329) (xy 181.5 73.201) (xy 181.749441 73.033329)
+				(xy 183.25 82.194236) (xy 183.75 82.194236) (xy 183.794236 81.658527) (xy 183.5 81.599) (xy 183.205764 81.658527)
 			)
 		)
@@
 	)
 	(zone
-		(net 2)
-		(net_name "+9V")
+		(net 7)
+		(net_name "/MotorConnect2")
 		(layer "B.Cu")
 		(name "$teardrop_padvia$")
 		(hatch none 0.1)
-		(priority 30001)
+		(priority 30004)
 		(attr
 			(teardrop
@@
 		(polygon
 			(pts
-				(xy 193.422943 84.45) (xy 193.422943 84.95) (xy 194.058527 84.894236) (xy 194.001 84.6) (xy 193.941473 84.305764)
+				(xy 183.75 81.005764) (xy 183.25 81.005764) (xy 183.205764 81.541473) (xy 183.5 81.601) (xy 183.794236 81.541473)
 			)
 		)
 	)
 	(zone
-		(net 13)
-		(net_name "/Input1")
+		(net 20)
+		(net_name "/Input2")
 		(layer "B.Cu")
 		(name "$teardrop_padvia$")
 		(hatch none 0.1)
-		(priority 30005)
+		(priority 30006)
 		(attr
 			(teardrop
@@
 		(polygon
 			(pts
-				(xy 178.805764 93.0365) (xy 178.805764 93.1635) (xy 179.233329 93.349441) (xy 179.401 93.1) (xy 179.233329 92.850559)
+				(xy 181.07145 73.5365) (xy 181.07145 73.6635) (xy 181.558527 73.494236) (xy 181.501 73.2) (xy 181.205764 73.141473)
 			)
 		)
 	)
 	(zone
-		(net 2)
-		(net_name "+9V")
+		(net 13)
+		(net_name "/Input1")
 		(layer "B.Cu")
 		(name "$teardrop_padvia$")
 		(hatch none 0.1)
-		(priority 30002)
+		(priority 30005)
 		(attr
 			(teardrop
@@
 		(polygon
 			(pts
-				(xy 189.194236 84.95) (xy 189.194236 84.45) (xy 188.658527 84.405764) (xy 188.599 84.7) (xy 188.658527 84.994236)
+				(xy 178.805764 93.0365) (xy 178.805764 93.1635) (xy 179.233329 93.349441) (xy 179.401 93.1) (xy 179.233329 92.850559)
 			)
 		)
 	)
 	(zone
-		(net 7)
-		(net_name "/MotorConnect2")
+		(net 3)
+		(net_name "+3.3V")
 		(layer "B.Cu")
 		(name "$teardrop_padvia$")
 		(hatch none 0.1)
-		(priority 30004)
+		(priority 30003)
 		(attr
 			(teardrop
@@
 		(polygon
 			(pts
-				(xy 183.75 81.005764) (xy 183.25 81.005764) (xy 183.205764 81.541473) (xy 183.5 81.601) (xy 183.794236 81.541473)
+				(xy 191.905764 78.65) (xy 191.905764 79.15) (xy 192.441473 79.194236) (xy 192.501 78.9) (xy 192.441473 78.605764)
 			)
 		)
 	)
 	(zone
-		(net 3)
-		(net_name "+3.3V")
+		(net 1)
+		(net_name "GND")
+		(layer "B.Cu")
+		(hatch edge 0.5)
+		(connect_pads yes
+			(clearance 0.5)
+		)
+		(min_thickness 0.25)
+		(filled_areas_thickness no)
+		(fill yes
+			(thermal_gap 0.5)
+			(thermal_bridge_width 0.5)
+		)
+		(polygon
+			(pts
+				(xy 168.3 66.7) (xy 200.9 66.5) (xy 200.9 97.6) (xy 168.1 97.2)
+			)
+		)
+	)
+	(zone
+		(net 2)
+		(net_name "+9V")
 		(layer "B.Cu")
 		(name "$teardrop_padvia$")
 		(hatch none 0.1)
-		(priority 30003)
+		(priority 30001)
 		(attr
 			(teardrop
@@
 		(polygon
 			(pts
-				(xy 191.905764 78.65) (xy 191.905764 79.15) (xy 192.441473 79.194236) (xy 192.501 78.9) (xy 192.441473 78.605764)
+				(xy 193.422943 84.45) (xy 193.422943 84.95) (xy 194.058527 84.894236) (xy 194.001 84.6) (xy 193.941473 84.305764)
 			)
 		)
@@
 	)
 	(zone
-		(net 1)
-		(net_name "GND")
-		(layer "B.Cu")
-		(hatch edge 0.5)
-		(connect_pads yes
-			(clearance 0.5)
-		)
-		(min_thickness 0.25)
-		(filled_areas_thickness no)
-		(fill yes
-			(thermal_gap 0.5)
-			(thermal_bridge_width 0.5)
-		)
-		(polygon
-			(pts
-				(xy 168.3 66.7) (xy 200.9 66.5) (xy 200.9 97.6) (xy 168.1 97.2)
-			)
-		)
-	)
-	(zone
-		(net 20)
-		(net_name "/Input2")
+		(net 2)
+		(net_name "+9V")
 		(layer "B.Cu")
 		(name "$teardrop_padvia$")
 		(hatch none 0.1)
-		(priority 30006)
+		(priority 30002)
 		(attr
 			(teardrop
@@
 		(polygon
 			(pts
-				(xy 181.07145 73.5365) (xy 181.07145 73.6635) (xy 181.558527 73.494236) (xy 181.501 73.2) (xy 181.205764 73.141473)
+				(xy 189.194236 84.95) (xy 189.194236 84.45) (xy 188.658527 84.405764) (xy 188.599 84.7) (xy 188.658527 84.994236)
 			)
 		)

Commit message: Add files via upload
Parts:
- moved MotorLoad1 13.8 mm to (180.4, 78.3)
- moved C9 10.1 mm to (189.2, 69.7), turned to -90 degrees
- moved U8 9.78 mm to (193.7, 69.4), turned to 180 degrees
- moved C11 7.94 mm to (198.6, 84.2), turned to 90 degrees
- moved C6 7.40 mm to (196.7, 74.2)
- moved U4 7.40 mm to (193.4, 74.2)
- moved U5 7.40 mm to (185.9, 74.2)
- moved C7 7.40 mm to (188.9, 74.1)
- moved Q3 6.48 mm to (192.5, 78.7)
- moved Q4 6.48 mm to (187.2, 78.9)
- moved C10 6.40 mm to (197.3, 86.8)
- moved U7 6.19 mm to (187.1, 69.4), turned to 0 degrees
- moved C2 5.04 mm to (191.5, 70.7), turned to -90 degrees
- moved 9VPower1 2.65 mm to (195.6, 92.2), turned to -90 degrees
- moved C3 1.30 mm to (193.2, 89.4), turned to 0 degrees
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Routing:
- net +3.3V: track 40.1 -> 52.2 mm, vias 4 -> 2
- net /Input2: track 19.9 -> 32.0 mm, vias 1 -> 2
- net /MotorConnect2: track 20.7 -> 10.00 mm, vias 1 -> 0
- net /Enable: track 34.6 -> 43.6 mm
- net +9V: track 16.2 -> 8.77 mm, vias 2 -> 0
- net /MotorConnect1: track 20.1 -> 13.7 mm
- net Net-(U4-Pad1): track 1.82 -> 6.49 mm, vias 0 -> 2
- net Net-(U5-Pad1): track 8.92 -> 4.98 mm
- net GND: track 28.0 -> 26.2 mm, vias 16 -> 17
- net Net-(Q4-G): track 4.25 -> 5.55 mm, vias 0 -> 2
- net Net-(U10-BYP): track 2.51 -> 3.19 mm

Commit message: final revisions for layout
Parts:
- added G***: LOGO, Logo:ElectriumLogo, F.Cu at (175.7, 71.5)
- added H1: MountingHole, MountingHole:MountingHole_2.5mm, F.Cu at (172.0, 93.5)
Other:
- board size 30.4 x 28.7 mm -> 30.5 x 29 mm
- board text added: "Eleanor"

Commit message: Add files via upload
Parts:
- moved U7 0.43 mm to (187.1, 69.8)
- moved C9 0.33 mm to (189.2, 70.0)
Routing:
- net +3.3V: track 52.2 -> 58.6 mm, vias 2 -> 0
- net /Input2: track 32.0 -> 33.5 mm
- net GND: track 26.2 -> 27.4 mm, vias 17 -> 18
- net Net-(U4-Pad1): track 6.49 -> 7.44 mm
- net Net-(U1-Pad4): track 7.34 -> 6.76 mm
- net /Input1: track 17.5 -> 17.3 mm, vias 1 -> 0
Other:
- board text added: "En"
- board text added: "In1"
- board text added: "In2"
- board text added: "M1"
- board text added: "M2"
- board text removed: "Enable"
- board text removed: "Input1"
- board text removed: "Input2"
- board text removed: "Motor1"
- board text removed: "Motor2"
